File: RC/RC KiCAD/_autosave-RC KiCAD.kicad_sch (KiCad schematic)
At the start: 2 parts, among them J1 CX90B1-24P

Commit message: Uploading new RC PCB Components
Parts:
- added BT1: 1043P, 1043P:BAT_1043P, symbol 1043P:1043P
- added C2: JMK325ABJ107MM-P, JMK325ABJ107MM-P:CAPC3225X280N, symbol JMK325ABJ107MM-P:JMK325ABJ107MM-P
- added R13: CRM2512-FX-2R00ELF, CRM2512-FX-2R00ELF:RESC6331X80N, symbol CRM2512-FX-2R00ELF:CRM2512-FX-2R00ELF
- added R15: RMCF2512JT3K30, RMCF2512JT3K30:RESC6332X70N, symbol RMCF2512JT3K30:RMCF2512JT3K30
- added R16: CRCW12101K40FKEA, CRCW12101K40FKEA:RESC3225X60N, symbol CRCW12101K40FKEA:CRCW12101K40FKEA
- added VR1, VR2: LM317T, LM317T:TO254P1054X470X1955-3, symbol LM317T:LM317T
Connections:
- net BMS VCC: now also VR1.3 (VIN)
- net GND: no longer C1.2
- new net: C2.1, R16.1, VR1.2 (VOUT), VR2.3 (VIN)
- new net: R15.1, R16.2, VR1.1 (ADJ)
- new net: C1.2, C2.2, R15.2
- new net: BT1.P, R13.2, VR2.1 (ADJ)
- new net: R13.1, VR2.2 (VOUT)
Other:
- moved on the sheet: C1

Commit message: Adding more components
Parts:
- added Q2: BD140, BD140:TO229P760X270X1364-3, symbol BD140:BD140
- added R1, R2, R4: RMCF1206FT20R0, RMCF1206FT20R0:RESC3216X70N, symbol RMCF1206FT20R0:RMCF1206FT20R0
- added R3: RMCF1206FT1K00, RMCF1206FT1K00:RESC3216X70N, symbol RMCF1206FT1K00:RMCF1206FT1K00
- added U1: TL431AIDBZR, TL431AIDBZR:SOT95P237X112-3N, symbol TL431AIDBZR:TL431AIDBZR
Connections:
- net at BT1.N: now also R4.2, U1.1 (REF)
- net at BT1.P, R13.2, VR2.1 (ADJ): now also Q2.1, R2.1, R3.1
- new net: R1.2, R4.1
- new net: Q2.3, R3.2, U1.2 (CATHODE)
- new net AN: R1.1, R2.2, U1.3 (ANODE)

Commit message: BMS FULL CAO
Parts:
- added BT2: 1043P, Footprints:BAT_1043P, symbol 1043P:1043P
- added D1, D2, D3, D4: DSS14UTR, DSS14UTR:SODFL3618X110N, symbol DSS14UTR:DSS14UTR
- added LED1: APT1608SGC, Footprints:LED_APT1608SGC_KNB, symbol APT1608SGC:APT1608SGC
- added R4: RMCF2512JT330R, RMCF2512JT330R:RESC6332X70N, symbol RMCF2512JT330R:RMCF2512JT330R
- C1, C2: footprint JMK325ABJ107MM-P:CAPC3225X280N -> Footprints:CAPC3225X280N
- J1: footprint CX90B1-24P:HRS_CX90B1-24P -> Footprints:HRS_CX90B1-24P
- Q2: footprint BD140:TO229P760X270X1364-3 -> Footprints:TO229P760X270X1364-3
- R13: footprint CRM2512-FX-2R00ELF:RESC6331X80N -> Footprints:RESC6331X80N
- U12: renamed from VR1; footprint LM317T:TO254P1054X470X1955-3 -> Footprints:TO254P1054X470X1955-3
- U6: renamed from VR2; footprint LM317T:TO254P1054X470X1955-3 -> Footprints:TO254P1054X470X1955-3
- renumbered R4 to R10
Connections:
- net GND: now also C1.2, C2.2, R10.2, R15.2, U1.1 (REF), BT2.N, D4.C, LED1.2
- net at Q2.2: now also D1.A, R4.1
- new net: LED1.1, R4.2
- new net: D2.C, D3.A
- new net: D3.C, D4.A
- new net: BT1.N, BT2.P
- new net: D1.C, D2.A
Other:
- moved on the sheet: BT1
