File: RC/RC KiCAD/RC KiCAD.kicad_sch (KiCad schematic)
At the start: 22 parts, among them J1 CX90B1-24P, Q2 BD140, U1 TL431AIDBZR, U12 LM317T, U6 LM317T

Commit message: New components added
Parts:
- removed J1: CX90B1-24P, Footprints:HRS_CX90B1-24P, symbol CX90B1-24P:CX90B1-24P
- added BOOT_SW, RESET_SW: PTS810_SJM_250_SMTR_LFS, Footprints:SW_PTS810_SJM_250_SMTR_LFS, symbol PTS810_SJM_250_SMTR_LFS:PTS810_SJM_250_SMTR_LFS
- added C3, C5, C6: 0.1uF, symbol Device:C_Small
- added C4, C7, C8: 10uF, symbol Device:C_Small
- added D5: WS2812B, LED_SMD:LED_WS2812B_PLCC4_5.0x5.0mm_P3.2mm, symbol LED:WS2812B
- added D6: LED, LED_SMD:LED_0603_1608Metric, symbol Device:LED
- added J1: USB4085, Footprints:GCT_USB4085-GF-A_REVB, symbol USB4085-GF-A_REVB:USB4085-GF-A_REVB
- added LS1: CEM-1206S, Footprints:CUI_CEM-1206S, symbol CEM-1206S:CEM-1206S
- added R11, R5, R6: 5.1k, symbol Device:R_Small
- added R7: 10k, symbol Device:R_Small
- added R8: 1M, symbol Device:R_Small
- added R9: 200k, symbol Device:R_Small
- added S1: 400BWMSP1R2BLKSM6QE, Footprints:SW_400BWMSP1R2BLKSM6QE, symbol 400BWMSP1R2BLKSM6QE:400BWMSP1R2BLKSM6QE
- added U2: D3V3XA4B10LP, Package_DFN_QFN:Diodes_UDFN-10_1.0x2.5mm_P0.5mm, symbol Power_Protection:D3V3XA4B10LP
- added U3: ESP32-S3-WROOM-2-N32R8V, Footprints:XCVR_ESP32-S3-WROOM-2-N32R8V, symbol ESP32-S3-WROOM-2-N32R8V:ESP32-S3-WROOM-2-N32R8V
- added U4: TLV75801PDBV, Package_TO_SOT_SMD:SOT-23-5, symbol Regulator_Linear:TLV75801PDBV
Connections:
- net GND: now also BOOT_SW.1, BOOT_SW.2, C3.2, C4.2, C5.2, C6.2, C7.2, C8.2, D5.3 (VSS), D6.1 (K), J1.A1 (GND), J1.A12 (GND__1), J1.B1 (GND__2), J1.B12 (GND__3), J1.S1 (SHELL), J1.S2 (SHELL__1), J1.S3 (SHELL__2), J1.S4 (SHELL__3), LS1.N, R5.2, R6.2, R9.2, RESET_SW.1, RESET_SW.2, U2.3 (VSS), U2.8 (VSS), U4.2 (GND)
- net at BT1.P, Q2.1, R13.2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: now also S1.2
- net at C1.1, U12.3 (VIN): now also J1.A4 (VBUS), J1.A9 (VBUS__1), J1.B4 (VBUS__2), J1.B9 (VBUS__3)
- net AN renamed ANODE
- new net: D6.2 (A), R11.2
- new net: J1.A5 (CC1), R6.1
- new net: C3.1, C4.1, U3.2 (3V3)
- new net: R8.2, R9.1, U4.4 (FB)
- new net: BOOT_SW.3, BOOT_SW.4, C6.1, U3.27 (IO0)
- new net: LS1.P, U3.8 (IO15)
- new net: J1.B5 (CC2), R5.1
- new net 3V3: C8.1, D5.1 (VDD), R11.1, R7.1, R8.1, U4.5 (OUT)
- new net 5V USB: C7.1, S1.1, U2.4, U4.1 (IN), U4.3 (EN)
- new net D+: J1.A6 (DP1), J1.B6 (DP2), U2.1
- new net D-: J1.A7 (DN1), J1.B7 (DN2), U2.2
- new net ESP32_EN: C5.1, R7.2, RESET_SW.3, RESET_SW.4, U3.3 (EN)
- new net GPIO 48: D5.4 (DIN)
- new net RGB LED: U3.25 (IO48)
- no-connect marks 23 -> 2
Other:
- note added: "5V -> 4.2V"
- note added: "600mA limit"
- note added: "BMS PCB"
- note added: "CARP Alexandru"
- note added: "Linear Regulator"
- note added: "PWR LED"
- note added: "RGB LED"
- note removed: "25 Jun 2024"
- note removed: "ESP32-S3 PCB MainFrame"
- company: (none) -> CampusFab FabRice 
- title: (none) -> RC PCB 
- moved on the sheet: BT1, BT2, C1, C2, D1, D2, D3, D4, LED1, Q2, R1, R10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
