File: RC/RC KiCAD/_autosave-RC KiCAD.kicad_pcb (KiCad board)
At the start: 4 copper layers, 165 x 100 mm, 22 parts, among them J1 USB4125-GF-A_REVA2, Q2 BD140, U1 TL431AIDBZR, U12 LM317T, U6 LM317T

Commit message: autosave: new components added
Parts:
- added BOOT_SW1: PTS810_SJM_250_SMTR_LFS, Footprints:SW_PTS810_SJM_250_SMTR_LFS, B.Cu at (166.5, 31.5)
- added D5: WS2812B, LED_SMD:LED_WS2812B_PLCC4_5.0x5.0mm_P3.2mm, B.Cu at (71.5, 48.5)
- added D6: LED, LED_SMD:LED_0603_1608Metric, F.Cu at (137.5, 48.7)
- added H1: MountingHole_Pad, MountingHole:MountingHole_2.2mm_M2_Pad, F.Cu at (84.3, 82.7)
- added H2: MountingHole_Pad, MountingHole:MountingHole_2.2mm_M2_Pad, F.Cu at (58.3, 108.1)
- added H3: MountingHole_Pad, MountingHole:MountingHole_2.2mm_M2_Pad, F.Cu at (186.0, 26.6)
- added H4: MountingHole_Pad, MountingHole:MountingHole_2.2mm_M2_Pad, F.Cu at (165.8, 108.3)
- added J2: ~, Footprints:CON_524373071_MOL, F.Cu at (134.7, 101.0)
- added LS1: CEM-1206S, Footprints:CUI_CEM-1206S, B.Cu at (159.9, 61.1)
- added RESET_SW1: PTS810_SJM_250_SMTR_LFS, Footprints:SW_PTS810_SJM_250_SMTR_LFS, B.Cu at (166.6, 24.7)
- added S1: 400BWMSP1R2BLKSM6QE, Footprints:SW_400BWMSP1R2BLKSM6QE, B.Cu at (88.4, 29.1)
- added U2: D3V3XA4B10LP, Package_DFN_QFN:Diodes_UDFN-10_1.0x2.5mm_P0.5mm, F.Cu at (117.7, 43.7)
- added U3: ESP32-S3-WROOM-2-N32R8V, Footprints:XCVR_ESP32-S3-WROOM-2-N32R8V, F.Cu at (140.8, 32.9)
- added U4: TLV75801PDBV, Package_TO_SOT_SMD:SOT-23-5, F.Cu at (106.4, 27.9)
- J1: value USB4125-GF-A_REVA2 -> USB4085; footprint Footprints:GCT_USB4125-GF-A_REVA2 -> Footprints:GCT_USB4085-GF-A_REVB
- moved LED1 2.12 mm to (66.1, 21.3)
- moved J1 0.50 mm to (58.0, 21.3)
Connections:
- net AN renamed /ANODE
- net USB D+ renamed Net-(J1-CC1)
- net USB D- renamed Net-(J1-CC2)
Routing:
- net Net-(U6-ADJ): track 88.3 -> 144.0 mm, vias 1 -> 3
- net /ESP32_EN: track 0.00 -> 55.4 mm, vias 0 -> 2
- net Net-(U3-IO15): track 0.00 -> 52.3 mm, vias 0 -> 1
- net Net-(U3-IO0): track 0.00 -> 23.9 mm
- net GND: track 241.4 -> 247.8 mm
- net Net-(J1-VBUS): track 31.5 -> 37.2 mm
- net Net-(BT1-PadN): track 161.1 -> 156.7 mm
- net Net-(LED1-Pad1): track 2.91 -> 3.72 mm
- added copper zone on B.Cu, net GND
- removed copper zone on F.Cu, net GND
Other:
- copper layers 4 -> 2
