File: PCB_TELECOMANDE/RC KiCAD.kicad_sch (KiCad schematic)
At the start: 49 parts, among them J1 USB4085, Q2 BD140, U1 TL431AIDBZR, U12 LM317T, U2 D3V3XA4B10LP, U3 ESP32-S3-WROOM-2-N32R8V, U4 TLV75801PDBV, U6 LM317T

Commit message: Improving Charging efficency to 90%
Parts:
- removed BT1: 1043P, 1043P:BAT_1043P, symbol 1043P:1043P
- removed BT2: 1043P, Footprints:BAT_1043P, symbol 1043P:1043P
- removed C1, C2: JMK325ABJ107MM-P, Footprints:CAPC3225X280N, symbol JMK325ABJ107MM-P:JMK325ABJ107MM-P
- removed D1, D2, D3, D4: DSS14UTR, Footprints:SODFL3618X110N, symbol DSS14UTR:DSS14UTR
- removed LED1: APT1608SGC, Footprints:LED_APT1608SGC_KNB, symbol APT1608SGC:APT1608SGC
- removed Q2: BD140, Footprints:TO229P760X270X1364-3, symbol BD140:BD140
- removed R1, R10, R2: RMCF1206FT20R0, Footprints:RESC3216X70N, symbol RMCF1206FT20R0:RMCF1206FT20R0
- removed R13: CRM2512-FX-2R00ELF, Footprints:RESC6331X80N, symbol CRM2512-FX-2R00ELF:CRM2512-FX-2R00ELF
- removed R15: RMCF2512JT3K30, Footprints:RESC3216X70N, symbol RMCF2512JT3K30:RMCF2512JT3K30
- removed R16: CRCW12101K40FKEA, Footprints:RESC3225X60N, symbol CRCW12101K40FKEA:CRCW12101K40FKEA
- removed R3: RMCF1206FT1K00, Footprints:RESC3216X70N, symbol RMCF1206FT1K00:RMCF1206FT1K00
- removed R4: RMCF2512JT330R, Footprints:RESC6332X70N, symbol RMCF2512JT330R:RMCF2512JT330R
- removed S1: 400BWMSP1R2BLKSM6QE, Footprints:SW_400BWMSP1R2BLKSM6QE, symbol 400BWMSP1R2BLKSM6QE:400BWMSP1R2BLKSM6QE
- removed U1: TL431AIDBZR, Footprints:SOT95P237X112-3N, symbol TL431AIDBZR:TL431AIDBZR
- removed U12, U6: LM317T, Footprints:TO254P1054X470X1955-3, symbol LM317T:LM317T
- removed U2: D3V3XA4B10LP, Package_DFN_QFN:Diodes_UDFN-10_1.0x2.5mm_P0.5mm, symbol Power_Protection:D3V3XA4B10LP
- added C1, C10, C9: 0.1uF, symbol Device:C_Small
- added C2: 0.33uF, symbol Device:C_Small
- added CR1: SMF9.0CA, SOD-123F_LTF, symbol SMF9_0CA:SMF9.0CA
- added F1: Polyfuse_Small, symbol Device:Polyfuse_Small
- added F2: Fuse_Small, symbol Device:Fuse_Small
- added J4: BAT2_CON, 1990009:PHOENIX_1990009, symbol 1990009:1990009
- added J5: BAT1_CON, 1990009:PHOENIX_1990009, symbol 1990009:1990009
- added L1: 60R @ 100MHz, symbol Device:L_Small
- added Q1: PMV45EN2, Package_TO_SOT_SMD:SOT-23-3, symbol Simulation_SPICE:NMOS
- added R1, R2: 5.1K, symbol Device:R_Small
- added R10: 160, symbol Device:R_Small
- added R12: 0, TestPoint:TestPoint_2Pads_Pitch2.54mm_Drill0.8mm, symbol Device:R_Small
- added R3: 1k, symbol Device:R_Small
- added R4: 100, symbol Device:R_Small
- added TP1: GND, Connector_Pin:Pin_D1.0mm_L10.0mm, symbol Connector:TestPoint
- added TP2: VBUS, Connector_Pin:Pin_D1.0mm_L10.0mm, symbol Connector:TestPoint
- added TP3, TP5, TP7: TestPoint, symbol Connector:TestPoint
- added TP4: BAT1+, symbol Connector:TestPoint
- added TP6: BAT2+, symbol Connector:TestPoint
- added TP8: PACK-, symbol Connector:TestPoint
- added TP9: PACK+, symbol Connector:TestPoint
- added U1: BQ29200DRBT, BQ29200DRBT:IC_DRV8601DRBT, symbol BQ29200DRBT:BQ29200DRBT
- added U2: BQ24133RGYR, BQ24133RGYR:QFN50P550X350X100-25N, symbol BQ24133RGYR:BQ24133RGYR
- added U5: LM2623MM, LM2623MM:SOP65P490X110-8N, symbol LM2623MM:LM2623MM
- R5: value 5.1k -> 260; footprint Resistor_SMD:R_0805_2012Metric -> (none)
- R6: value 5.1k -> 100; footprint Resistor_SMD:R_0805_2012Metric -> (none)
Connections:
- net GND: now also C2.1, L1.1, U1.5 (GND), U1.9 (EPAD); no longer J1.A1 (GND), J1.A12 (GND__1), J1.B1 (GND__2), J1.B12 (GND__3), J1.S1 (SHELL), J1.S2 (SHELL__1), J1.S3 (SHELL__2), J1.S4 (SHELL__3), R5.2, R6.2
- net at J1.A5 (CC1): now also R1.1; no longer R6.1
- net at J1.A4 (VBUS), J1.A9 (VBUS__1), J1.B4 (VBUS__2)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: now also TP2.1
- net at R5.1: now also R6.1, J4.1, J5.2, TP4.1, TP7.1; no longer J1.B5 (CC2)
- new net: F2.1, J4.2, R10.1, R12.1, R4.2, TP6.1
- new net: CR1.1, F1.2, TP3.1
- new net: Q1.1 (D), R12.2
- new net: Q1.2 (G), R3.2
- new net: J1.B5 (CC2), R2.1
- new net: C1.1, R4.1, U1.7 (VDD)
- new net: R3.1, U1.8 (OUT)
- new net: C9.1, R10.2
- new net: C10.1, C9.2, R5.2
- new net GNDREF: CR1.2, J1.A1 (GND), J1.A12 (GND__1), J1.B1 (GND__2), J1.B12 (GND__3), J1.S1 (SHELL), J1.S2 (SHELL__1), J1.S3 (SHELL__2), J1.S4 (SHELL__3), L1.2, R1.2, R2.2, TP1.1
- new net PACK+: F2.2, TP9.1
- new net PACK-: C1.2, C10.2, J5.1, Q1.3 (S), TP5.1, TP8.1
- no-connect marks 36 -> 30
Other:
- note added: "BATTERY PROTECTION SYSTEM"
- note added: "USB"
- note removed: "5V -> 4.2V"
- note removed: "600mA limit"
- note removed: "BMS PCB"
- note removed: "CARP Alexandru"
- moved on the sheet: BOOT_SW1, C3, C4, C5, C6, C7, C8, D5, D6, H1, H2, H3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

Commit message: Filesys Reorg + PD Negociator schematics
Parts:
- removed TP1: GND, Connector_Pin:Pin_D1.0mm_L10.0mm, symbol Connector:TestPoint
- removed U5: LM2623MM, LM2623MM:SOP65P490X110-8N, symbol LM2623MM:LM2623MM
- added C11, C12: 0.1uF, symbol Device:C_Small
- added C13, C15, C16, C19: 4.7uF, symbol Device:C_Small
- added C14, C17, C18, C20: 100nF, symbol Device:C_Small
- added D1: ESDA25W, ESDA25W:SOT65P210X110-3N, symbol ESDA25W:ESDA25W
- added D2: BAT60A, Diode_SMD:D_SOD-323, symbol Diode:BAT60A
- added D3: LED, LED_SMD:LED_0603_1608Metric, symbol Device:LED
- added MOSFET1, MOSFET2: DMP3098LQ-7, SOT-23_DMP3098LQ_DIO, symbol DMP3098LQ_7:DMP3098LQ-7
- added Q2: 2N7002K-7, 2N7002K-7:SOT91P240X110-3N, symbol 2N7002K-7:2N7002K-7
- added R13, R14, R15: 100K, symbol Device:R_Small
- added R16, R17, R19, R20, R21, R22, R23, R24, R25, R26, R27, R28, R29, R30, R31: 2.2k, symbol Device:R_Small
- added R18, R32: 20k, symbol Device:R_Small
- added RESET_SW2: PTS810_SJM_250_SMTR_LFS, Footprints:SW_PTS810_SJM_250_SMTR_LFS, symbol PTS810_SJM_250_SMTR_LFS:PTS810_SJM_250_SMTR_LFS
- added U5: STUSB4500QTR, STUSB4500QTR:QFN50P400X400X90-25N, symbol STUSB4500QTR:STUSB4500QTR
- added U6: CYPD3177-24LQ, Package_DFN_QFN:QFN-24-1EP_4x4mm_P0.5mm_EP2.75x2.75mm, symbol Interface_USB:CYPD3177-24LQ
- R1, R2: value 5.1K -> R_Small
- TP3: footprint (none) -> TestPoint:TestPoint_Pad_D1.5mm
Connections:
- net 3V3: now also C16.2, C17.1, C18.1, U6.23 (VDDD)
- net GND: now also C11.2, C12.2, C13.2, C14.2, C15.2, C16.1, C17.2, C18.2, D1.3, Q2.2, R13.2, R14.1, R15.1, R17.1, R21.1, R24.1, R25.1, R32.1, U5.10 (GND), U5.25 (EP)
- net GNDREF: no longer R1.2, R2.2
- net at R1.1: now also R2.1; no longer J1.A5 (CC1)
- net VBUS_LOCAL: now reaches CR1.1, F1.2, TP3.1
- net VBUS_LOCAL: now also C13.1, C14.1, U6.18 (VBUS_IN)
- net CC2_USB: now reaches J1.B5 (CC2)
- net CC2_USB: now also U6.14 (CC2); no longer R2.1
- net VBUS_USB: now reaches J1.A4 (VBUS), J1.A9 (VBUS__1), J1.B4 (VBUS__2), J1.B9 (VBUS__3), TP2.1
- net VBUS_USB: now also F1.1
- new net: R1.2, R13.1
- new net: D1.2, U5.1 (CC1DB), U5.2 (CC1)
- new net: C11.1, U5.21 (VREG_1V2)
- new net: C12.1, D2.2 (A), U5.23 (VREG_2V7)
- new net: D1.1, U5.4 (CC2), U5.5 (CC2DB)
- new net: R15.2, RESET_SW2.3, RESET_SW2.4, U5.6 (RESET)
- new net: C19.1, C20.1, R18.2, R19.2, R20.1
- new net: R16.1, R17.2, U6.2 (VBUS_MAX)
- new net: MOSFET1.1 (G), R19.1
- new net: C19.2, MOSFET1.2 (S), R18.1
- new net: R29.2, U6.12 (HPI_SDA)
- new net: R30.2, U6.7 (~{HPI_INT})
- new net: C15.1, U6.24 (VCCD)
- new net: D3.1 (K), R31.2
- new net: R21.2, R22.1, U6.1 (VBUS_MIN)
- new net: RESET_SW2.1, RESET_SW2.2
- new net: R14.2, R2.2
- new net: R23.2, R24.2
- new net: R27.2, U6.10 (FLIP)
- new net: R28.2, U6.13 (HPI_SCL)
- new net: U6.19 (GND), U6.22 (GND), U6.25 (GND)
- new net: Q2.1, R32.2, U6.9 (FAULT)
- new net: R25.2, R26.2
- new net: MOSFET1.3 (D), MOSFET2.3 (D)
- new net: Q2.3, R31.1
- new net 15V_LOCAL: C20.2, MOSFET2.2 (S)
- new net 3V3_MCU: D3.2 (A), R16.2, R22.2, R23.1, R26.1, R27.1, R28.1, R29.1, R30.1
- new net CC1_USB: J1.A5 (CC1), U6.15 (CC1)
- new net ISKN_FINE: U6.6 (ISNK_FINE)
- new net ISNK_COARSE: U6.5 (ISNK_COARSE)
- new net VBUS_FET_EN: U6.3 (VBUS_FET_EN)
- new net VDC_OUT: U6.11 (VDC_OUT)
Other:
- note added: "ISNK_CRS = 3A"
- note added: "PD NEGOCIATOR"
- note added: "VMAX = 15V"
- note added: "VMIN = 15V"
- moved on the sheet: C7, C8, CR1, D5, D6, F1, H1, H2, H3, H4, R11, R8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

Commit message: New PCB_ROBOT filesys
Parts:
- removed C11, C12: 0.1uF, symbol Device:C_Small
- removed D1: ESDA25W, ESDA25W:SOT65P210X110-3N, symbol ESDA25W:ESDA25W
- removed D2: BAT60A, Diode_SMD:D_SOD-323, symbol Diode:BAT60A
- removed R1, R2: R_Small, symbol Device:R_Small
- removed R13, R14, R15: 100K, symbol Device:R_Small
- removed RESET_SW2: PTS810_SJM_250_SMTR_LFS, Footprints:SW_PTS810_SJM_250_SMTR_LFS, symbol PTS810_SJM_250_SMTR_LFS:PTS810_SJM_250_SMTR_LFS
- removed U5: STUSB4500QTR, STUSB4500QTR:QFN50P400X400X90-25N, symbol STUSB4500QTR:STUSB4500QTR
- added R33: 0, Resistor_SMD:R_0603_1608Metric, symbol Device:R_Small
- added R34: 0, Resistor_SMD:R_1210_3225Metric, symbol Device:R_Small
- added TP1: 15V_OUT, TestPoint:TestPoint_Pad_D1.5mm, symbol Connector:TestPoint
- C13: footprint (none) -> Capacitor_SMD:C_0805_2012Metric
- C14, C15, C16, C17, C18: footprint (none) -> Capacitor_SMD:C_0603_1608Metric
- D3: value LED -> USB_FAULT_LED
- F1: footprint (none) -> Fuse:Fuse_Bourns_MF-RG300
- J4, J5: footprint 1990009:PHOENIX_1990009 -> Footprints:PHOENIX_1990009
- Q2: footprint 2N7002K-7:SOT91P240X110-3N -> Footprints:SOT91P240X110-3N
- R16, R22: value 2.2k -> 5.1k; footprint (none) -> Resistor_SMD:R_0603_1608Metric
- R17, R21: value 2.2k -> 2.4k; footprint (none) -> Resistor_SMD:R_0603_1608Metric
- R23, R24, R25, R26, R27, R28, R29, R30, R31: footprint (none) -> Resistor_SMD:R_0603_1608Metric
- TP4, TP5, TP6, TP7: footprint (none) -> TestPoint:TestPoint_Pad_D1.5mm
Connections:
- net 15V_LOCAL is gone; now on net VDC_OUT: C20.2, MOSFET2.2 (S)
- net 3V3_MCU: now also R33.2; no longer D3.2 (A), R27.1, R28.1, R29.1, R30.1
- net GND: now also U6.19 (GND), U6.22 (GND), U6.25 (GND)
- net ISKN_FINE: now also R25.2, R26.2
- net ISNK_COARSE: now also R23.2, R24.2
- net VDC_OUT: now also R34.1, TP1.1
- net VBUS_MOSFET: now reaches C19.2, MOSFET1.2 (S), R18.1
- net VC1_CB: now reaches R6.2
- net VC2: now reaches C9.1, R10.2
- net VC1: now reaches C10.1, C9.2, R5.2
- new net: D3.2 (A), R27.1, R28.1, R29.1, R30.1, R33.1
- new net 15V_OUT: R34.2
- no-connect marks 30 -> 32
Other:
- moved on the sheet: U2
