File: PCB_ROBOT/LAYER_0 - PWD/_autosave-LAYER_0 - PWD.kicad_sch (KiCad schematic)
At the start: 67 parts, among them J1 PRIMARY IN, J2 5031590600, J3 12V_IN, J4 5V_IN, Q1 CSD19534Q5A, Q2 CSD19532KTTT, U1 ACS712ELCTR-05B-T, U2 TPS566247DRLR, U3 LM5146RGYR

Commit message: temp save/ partial traces prog
Parts:
- removed J2: 5031590600, Footprints:CON_5031590600_MOL, symbol 5031590600:5031590600
- removed L1: 2.2uH, symbol Device:L
- added C23, C24, C25: 22uF, Capacitor_SMD:C_0805_2012Metric, symbol Device:C_Small
- added J5: V_I_SENSE, Footprints:17352658, symbol 1735265-8:1735265-8
- added L3: XAL5030-222MEC, XAL5030222MEC, symbol XAL5030-222MEC:XAL5030-222MEC
- added TP2: VSENSE_1, TestPoint:TestPoint_Pad_D1.5mm, symbol Connector:TestPoint
- C20, C21, C22: footprint (none) -> Capacitor_SMD:C_1210_3225Metric
- C4, C5, C7: footprint (none) -> Capacitor_SMD:C_0805_2012Metric
- C6, R19, R6, R7, R8, R9: footprint (none) -> Resistor_SMD:R_0603_1608Metric
- C8: footprint (none) -> Capacitor_SMD:C_0603_1608Metric
- Q1: footprint CSD19534Q5A:TRANS_CSD19534Q5A -> Footprints:TRANS_CSD19534Q5A
- TP1: value TestPoint -> ISENSE_1
Connections:
- net 12V_LOCAL is gone; now on net 12V_IN_5V_CONV: J3.1, R1.1
- net 56V_PROTECTED: now also J5.2, TP2.1
- net 5V_5A: now also C23.1, C24.1, C25.1, L3.2
- net GND: now also C23.2, C24.2, C25.2, J5.MP1, J5.MP2
- net ISENSE_1: now also J5.1
- net at U2.2 (SW): now also L3.1
Other:
- note added: "TRANSFORMER 12V"
- moved on the sheet: C10, C11, C12, C13, C14, C15, C16, C17, C18, C19, C20, C21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
